File: pcb/PLC_Output_PCB.kicad_sch (KiCad schematic)
At the start: 29 parts, among them J1 Conn_01x01_Socket, J2 Conn_01x01_Socket, J3 Conn_01x01_Socket, J4 Conn_01x01_Socket, J5 Conn_01x01_Socket, J6 Conn_01x01_Socket, J7 Conn_01x01_Socket, J8 Conn_01x01_Socket, K1 SANYOU_SRD_Form_C, K2 SANYOU_SRD_Form_C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

Commit message: Started PCB
Parts:
- removed J1, J2, J3, J4, J5, J6, J7, J8: Conn_01x01_Socket, Connector_PinSocket_1.00mm:PinSocket_1x02_P1.00mm_Vertical, symbol Connector:Conn_01x01_Socket
- added J10: Conn_01x08_Socket, Connector_PinSocket_1.00mm:PinSocket_1x08_P1.00mm_Vertical, symbol Connector:Conn_01x08_Socket
- added J9: Conn_01x01_Pin, Connector_PinHeader_1.00mm:PinHeader_1x01_P1.00mm_Vertical, symbol Connector:Conn_01x01_Pin
- R1: renamed from R3; footprint (none) -> Resistor_THT:R_Axial_DIN0207_L6.3mm_D2.5mm_P7.62mm_Horizontal_CUSTOM
- R10, R11, R12, R2, R4, R5, R6, R7, R8, R9: footprint (none) -> Resistor_THT:R_Axial_DIN0207_L6.3mm_D2.5mm_P7.62mm_Horizontal_CUSTOM
- R3: renamed from R1; footprint (none) -> Resistor_THT:R_Axial_DIN0207_L6.3mm_D2.5mm_P7.62mm_Horizontal_CUSTOM
Connections:
- net GND is gone; now on an unnamed net: R12.2, R3.2, R6.2, R9.2
- net COM: now also J9.1 (Pin_1)
- net at K6.3: now also J10.6 (Pin_6)
- net at K4.3: now also J10.4 (Pin_4)
- net at K1.3: now also J10.1 (Pin_1)
- net at K7.3: now also J10.7 (Pin_7)
- net at K8.3: now also J10.8 (Pin_8)
- net at K3.3: now also J10.3 (Pin_3)
- net at K2.3: now also J10.2 (Pin_2)
- net at K5.3: now also J10.5 (Pin_5)
